File: pcb/KiCad/PlexFlex/PlexFlex.kicad_pcb (KiCad board)
At the start: 2 copper layers, 298.7 x 6.7 mm, 2 parts

Commit message: Updated library locations, etc.
a79040_breakout: submitted to 4pcb.com for production.

PlexFlex: Still working.
Other:
- board size 298.7 x 6.7 mm -> 294.8 x 6.7 mm
Changed lines of the file:
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@@
     (links 18)
     (no_connects 0)
-    (area 37.338 64.643 336.55 77.724)
+    (area 30.125599 36.8274 329.081201 49.7636)
     (thickness 1.6)
     (drawings 4)
@@
     (visible_elements FFFFFF7F)
     (pcbplotparams
-      (layerselection 0x00030_80000001)
+      (layerselection 0x010a8_80000001)
       (usegerberextensions false)
-      (excludeedgelayer true)
+      (excludeedgelayer false)
       (linewidth 0.100000)
       (plotframeref false)
@@
       (psnegative false)
       (psa4output false)
-      (plotreference true)
-      (plotvalue true)
+      (plotreference false)
+      (plotvalue false)
       (plotinvisibletext false)
       (padsonsilk false)
@@
       (outputformat 1)
       (mirror false)
-      (drillshape 1)
+      (drillshape 0)
       (scaleselection 1)
-      (outputdirectory ""))
+      (outputdirectory plot))
   )
   (net 0 "")
@@
       (net 11 "Net-(REF1-Pad11)"))
   )
-  (gr_line (start 329.0316 46.6852) (end 329.0316 40.005) (angle 90) (layer Edge.Cuts) (width 0.15))
-  (gr_line (start 30.3022 46.736) (end 329.0316 46.736) (angle 90) (layer Edge.Cuts) (width 0.15))
-  (gr_line (start 30.3022 40.005) (end 30.3022 46.7106) (angle 90) (layer Edge.Cuts) (width 0.15))
-  (gr_line (start 30.3022 40.005) (end 329.0316 40.005) (angle 90) (layer Edge.Cuts) (width 0.15))
+  (gr_line (start 32.131 46.736) (end 326.898 46.736) (angle 90) (layer Edge.Cuts) (width 0.15))
+  (gr_line (start 326.898 40.005) (end 32.131 40.005) (angle 90) (layer Edge.Cuts) (width 0.15))
+  (gr_line (start 326.9234 40.0304) (end 326.9234 46.736) (angle 90) (layer Edge.Cuts) (width 0.15))
+  (gr_line (start 32.131 40.0304) (end 32.131 46.736) (angle 90) (layer Edge.Cuts) (width 0.15))
   (segment (start 35.6362 46.228) (end 323.5706 46.228) (width 0.127) (layer F.Cu) (net 1))
   (segment (start 323.5706 45.593) (end 323.2531 45.9105) (width 0.127) (layer F.Cu) (net 2))

Commit message: Add microphone: knowles_sph1642ht5h-1_revB - Footprint - Schematic - Add to flex cable design
Parts:
- added C1: omnetics_a79040, ugly:a79040, F.Cu at (325.7, 35.3)
- added U1: microphone_knowles_sph1642ht5h-1_revB, ugly:microphone_knowles_sph1642ht5h-1_revB, F.Cu at (34.9, 36.8)
Routing:
- net Net-(C1-Pad10): track 0.00 -> 295.4 mm
- net Net-(C1-Pad12): track 0.00 -> 289.6 mm
- net Net-(C1-Pad11): track 0.00 -> 288.8 mm
Other:
- board size 294.8 x 6.7 mm -> 294.8 x 14.8 mm
